Commit message: chore: phase 2 — vendor meshes into perseus_lite_description
Copies six meshes from perseus_description into perseus_lite_description
and repoints xacro references so the lite description is self-contained:

  chassis.dae, flange_bearing.dae, differential_bar.dae,
  rocker_left.dae, rocker_right.dae, gearbox.dae

Updated:
  - chassis.urdf.xacro, rocker.urdf.xacro, motor_wheel.urdf.xacro
    swap $(find perseus_description) for $(find perseus_lite_description)
  - package.xml drops <depend>perseus_description</depend>

With the dependency gone, perseus_description joins the COLCON_IGNORE
list. Workspace builds clean with 15 packages; resolved URDF has 18
mesh references, zero stale perseus_description paths.

File: software/ros_ws/src/perseus_lite_description/urdf/chassis.urdf.xacro (robot description, xacro)
@@ -16,5 +16,5 @@
         <origin xyz="0.0 0.0 0.0" rpy="0 0.0 ${-pi/2}"/>
         <geometry>
-          <mesh scale="0.05 0.05 0.05" filename="file://$(find perseus_description)/meshes/chassis.dae"/>
+          <mesh scale="0.05 0.05 0.05" filename="file://$(find perseus_lite_description)/meshes/chassis.dae"/>
         </geometry>
       </visual>
@@ -37,5 +37,5 @@
         <origin xyz="0.0 0.0 0.0" rpy="0 0 0"/>
         <geometry>
-          <mesh scale="0.05 0.05 0.05" filename="file://$(find perseus_description)/meshes/flange_bearing.dae"/>
+          <mesh scale="0.05 0.05 0.05" filename="file://$(find perseus_lite_description)/meshes/flange_bearing.dae"/>
         </geometry>
       </visual>
@@ -43,5 +43,5 @@
         <origin xyz="0.0 0.0 0.0" rpy="0 0 0"/>
         <geometry>
-          <mesh scale="0.05 0.05 0.05" filename="file://$(find perseus_description)/meshes/flange_bearing.dae"/>
+          <mesh scale="0.05 0.05 0.05" filename="file://$(find perseus_lite_description)/meshes/flange_bearing.dae"/>
         </geometry>
       </collision>
@@ -63,5 +63,5 @@
         <origin xyz="0.0 0.0 0.0" rpy="0.0 0.0 0.0"/>
         <geometry>
-          <mesh scale="0.05 0.05 0.05" filename="file://$(find perseus_description)/meshes/differential_bar.dae"/>
+          <mesh scale="0.05 0.05 0.05" filename="file://$(find perseus_lite_description)/meshes/differential_bar.dae"/>
         </geometry>
       </visual>

File: software/ros_ws/src/perseus_lite_description/urdf/motor_wheel.urdf.xacro (robot description, xacro)
@@ -13,5 +13,5 @@
         <origin xyz="-0.0 0.0 0.0" rpy="0.0 0.0 ${pi/2}"/>
         <geometry>
-          <mesh scale="0.05 0.05 0.05" filename="file://$(find perseus_description)/meshes/gearbox.dae"/>
+          <mesh scale="0.05 0.05 0.05" filename="file://$(find perseus_lite_description)/meshes/gearbox.dae"/>
         </geometry>
         <!-- <material name="white"/> -->

File: software/ros_ws/src/perseus_lite_description/urdf/rocker.urdf.xacro (robot description, xacro)
@@ -20,5 +20,5 @@
         <origin xyz="0.0 0.0 0.0" rpy="0.0 0.0 ${pi}"/>
         <geometry>
-          <mesh scale="0.05 0.05 0.05" filename="file://$(find perseus_description)/meshes/rocker_${side}.dae"/>
+          <mesh scale="0.05 0.05 0.05" filename="file://$(find perseus_lite_description)/meshes/rocker_${side}.dae"/>
         </geometry>
       </visual>
