Commit message: fix(perseus_lite): port the robot-validated drive/nav stack and one TF/velocity contract
Bring main in line with the configuration validated on the robot
(origin/feat/perseus-lite) and make hardware, simulation and Nav2 agree on
frames and topics:

- Controller: calibrated wheel_separation 0.8286 / wheel_radius 0.0725,
  velocity-feedback odometry, enable_odom_tf false (the EKF owns
  odom->base_link), conservative velocity/accel limits; dead hardware block
  and jsb effort mapping removed.
- URDF: lidar mounted centred under the chassis, upside down (as built).
- Bringup now starts the RPLidar C1, scan_range_filter (/scan ->
  /scan_filtered, drops the robot's own rockers/wheels inside 0.5 m), the
  robot_localization EKF, twist_mux (joy 100 > key 90 > web 80 > nav 10,
  output remapped to /cmd_vel) and rosbridge. Previously nothing published
  odom->base_link off-controller and twist_mux never reached the controller.
- One Nav2 launch (autonomy/perseus_nav_bringup) shared by the SLAM+Nav2,
  map-localisation, autonomy and mission launches: no phantom composition
  container, no bogus docking server, optional map_server+AMCL mode.
  perseus_lite_slam_and_nav2/nav2 now include the bringup instead of
  duplicating Nav2 and running a second EKF and AMCL alongside SLAM.
- Nav2 params: robot-tuned values, polygon footprint, /scan_filtered with a
  0.5 m min range, odometry/filtered, through-poses BT from perseus_bt_nodes,
  collision monitor zones that can actually see past the blind radius.
- slam_toolbox: base_link + /scan_filtered with the robot's CPU tuning; the
  mapping launch activates the lifecycle node instead of faking map->odom
  with a static TF.
- Simulation: shares perseus_lite's EKF, twist_mux and scan filter; EKF on
  by default; IMU bridged on imu/data; dead tf/odom/joint_state/Livox
  bridges removed.
- Remove unused v2-era autonomy configs and launches.

File: software/ros_ws/src/perseus_lite_description/urdf/sensors.urdf.xacro (robot description, xacro)
@@ -27,5 +27,6 @@
         <parent link="${prefix}chassis"/>
         <child link="${prefix}c1_lidar_frame"/>
-        <origin xyz="0.0 0.22 0.0" rpy="0 0 0"/>
+        <!-- Centred under the chassis and mounted upside down (as on the robot) -->
+        <origin xyz="0.0 0.0 -0.04" rpy="${pi} 0 0"/>
     </joint>
     <gazebo reference="${prefix}c1_lidar_frame">
