Commit message: fix(perseus_lite_hardware): port robot-validated ST3215 fixes and stop servos on faults
Brings the fixes proven on the physical robot (origin/feat/perseus-lite
4de13298, be17e49b, 656b28de, ff98e260) into main's refactored driver and
closes the remaining review findings:

- Stamp and check feedback with std::chrono::steady_clock. The ROS-time
  stamp was subtracted from the controller manager's steady clock, which
  throws, so the component dropped out on the first read().
- Negate feedback for inverted (left-side) servos, mirroring the command
  inversion; odometry previously saw the left wheels turning backward.
- Use the calibrated wheel-mode speed scale (full scale 32767 =
  servo_max_rpm, default 485.1, exposed as a hardware param). The old
  +/-1000 clamp capped each wheel at ~0.06 m/s.
- Unwrap wheel-mode position (0-4095 per revolution) into a continuous
  joint angle.
- Only a full status reply refreshes a servo's timestamp; WRITE ACKs are
  flushed before each status request and accumulated replies are parsed.
- Zero goal speed before enabling torque at configure; probe each servo;
  write zero speed + torque-off on cleanup/shutdown/on_error; catch
  std::exception (bad baud_rate) and close the port on configure failure.
- Set ACC=0 (no servo ramp) as on the robot, configurable.
- Flip the left wheel joint axis so positive joint velocity drives every
  wheel forward (+Y axis in base_link); sim previously spun in place.
- Add pty-backed system tests (fake servo bus) for lifecycle, inversion,
  unwrap, ACK staleness, missing servos and error stops; update protocol
  tests for the new scale. README rewritten (baud, IDs, safety behaviour).

File: software/ros_ws/src/perseus_lite/urdf/perseus_lite.urdf.xacro (robot description, xacro)
@@ -5,4 +5,5 @@
   <xacro:arg name="serial_port" default="/dev/ttyACM0" />
   <xacro:arg name="baud_rate" default="1000000" />
+  <xacro:arg name="servo_max_rpm" default="485.1" />
   <xacro:arg name="use_sim" default="false" />
   <!-- Import URDF description -->
@@ -19,5 +20,6 @@
     hardware_plugin="$(arg hardware_plugin)"
     serial_port="$(arg serial_port)"
-    baud_rate="$(arg baud_rate)"/>
+    baud_rate="$(arg baud_rate)"
+    servo_max_rpm="$(arg servo_max_rpm)"/>
   <!-- In simulation, gz_ros2_control hosts the controller_manager itself via
        this plugin tag; on real hardware controller_manager is launched as a

File: software/ros_ws/src/perseus_lite_description/ros2_control/perseus_lite.ros2_control.xacro (robot description, xacro)
@@ -1,5 +1,5 @@
 <?xml version="1.0"?>
 <robot xmlns:xacro="http://www.ros.org/wiki/xacro">
-  <xacro:macro name="perseus_lite_ros2_control" params="name prefix hardware_plugin serial_port baud_rate inverted_servo_ids:='2,3'">
+  <xacro:macro name="perseus_lite_ros2_control" params="name prefix hardware_plugin serial_port baud_rate inverted_servo_ids:='2,3' servo_max_rpm:='485.1' acceleration:='0'">
     <ros2_control name="${name}" type="system">
       <hardware>
@@ -9,4 +9,10 @@
         <!-- Left-side servos drive mirrored, so their velocity is inverted -->
         <param name="inverted_servo_ids">${inverted_servo_ids}</param>
+        <!-- RPM represented by a full-scale (32767) wheel-mode speed value.
+             485.1 was calibrated on the robot by comparing commanded and
+             measured wheel rotation; re-measure if servos are swapped. -->
+        <param name="servo_max_rpm">${servo_max_rpm}</param>
+        <!-- Servo ACC register: 0 disables the on-servo speed ramp -->
+        <param name="acceleration">${acceleration}</param>
       </hardware>
       <joint name="${prefix}front_left_wheel_joint">

File: software/ros_ws/src/perseus_lite_description/urdf/wheel.urdf.xacro (robot description, xacro)
@@ -24,6 +24,10 @@
     <!-- WHEEL -->
     <joint name="${prefix}${end}_${side}_wheel_joint" type="continuous">
+      <!-- Positive joint velocity must roll every wheel forward (+X of
+           base_link), i.e. the axis is +Y in base_link on both sides, as
+           diff_drive_controller assumes. The left motor link is yawed by pi,
+           so its local axis is flipped relative to the right side. -->
       <xacro:if value="${side == 'left'}">
-        <axis xyz="0 0 -1"/>
+        <axis xyz="0 0 1"/>
       </xacro:if>
       <xacro:if value="${side == 'right'}">
